Commit message: depth camera and mobile manipulator control ready

File: mobile_manipulator_description/urdf/mobile_manipulator.urdf.xacro (robot description, xacro)
@@ -3,4 +3,7 @@
   <xacro:include filename="$(find mobile_manipulator_description)/urdf/tracer_base.urdf.xacro"/>
   <xacro:include filename="$(find mobile_manipulator_description)/urdf/xarm7.urdf.xacro"/>
+  <!-- Placeholder wrist-camera mount. Replace these with measured D455 extrinsics. -->
+  <xacro:property name="wrist_camera_xyz" value="0.035 0 0.025"/>
+  <xacro:property name="wrist_camera_rpy" value="0 0 0"/>
   <xacro:tracer_base/>
   <xacro:xarm7/>
@@ -58,3 +61,36 @@
     <origin xyz="0.149 0 0.444" rpy="0 0 0"/>
   </joint>
+  <link name="wrist_camera_link">
+    <visual>
+      <origin xyz="0 0 0" rpy="0 0 0"/>
+      <geometry>
+        <box size="0.090 0.025 0.025"/>
+      </geometry>
+      <material name="realsense_gray">
+        <color rgba="0.12 0.12 0.13 1"/>
+      </material>
+    </visual>
+    <collision>
+      <origin xyz="0 0 0" rpy="0 0 0"/>
+      <geometry>
+        <box size="0.090 0.025 0.025"/>
+      </geometry>
+    </collision>
+    <inertial>
+      <origin xyz="0 0 0" rpy="0 0 0"/>
+      <mass value="0.072"/>
+      <inertia ixx="0.0000066" ixy="0" ixz="0" iyy="0.0000492" iyz="0" izz="0.0000492"/>
+    </inertial>
+  </link>
+  <joint name="link_eef_to_wrist_camera" type="fixed">
+    <parent link="link_eef"/>
+    <child link="wrist_camera_link"/>
+    <origin xyz="${wrist_camera_xyz}" rpy="${wrist_camera_rpy}"/>
+  </joint>
+  <link name="wrist_camera_color_optical_frame"/>
+  <joint name="wrist_camera_link_to_color_optical_frame" type="fixed">
+    <parent link="wrist_camera_link"/>
+    <child link="wrist_camera_color_optical_frame"/>
+    <origin xyz="0 0 0" rpy="0 0 0"/>
+  </joint>
 </robot>
